Commit message: updated urdf

File: ros_project_ws/src/qbot_description/urdf/qbot.urdf (robot description, URDF)
Before this commit: robot qbot, 9 links, 8 joints
Links:
- added link lidar_link; visual cylinder length=0.05 radius=0.03
- link base_link: geometry collision cylinder length=0.109 radius=0.178; visual cylinder length=0.109 radius=0.178
- link camera_link: mass 0.1 -> None
- link caster_back_link: mass 0.2 -> None
- link caster_front_link: mass 0.2 -> None
- link imu_link: mass 0.1 -> None
- link sensor_mount_link: mass 0.3 -> None
- link wheel_left_link: geometry collision cylinder length=0.03 radius=0.05; visual cylinder length=0.03 radius=0.05
- link wheel_right_link: geometry collision cylinder length=0.03 radius=0.05; visual cylinder length=0.03 radius=0.05
Joints:
- added joint lidar_joint: type fixed, parent base_link, child lidar_link, origin xyz=0 0 0.12 rpy=0 0 0
- joint caster_back_joint: origin xyz=-0.135 0 0.009 rpy=-1.5708 0 0 -> xyz=-0.135 0 0.009
- joint caster_front_joint: origin xyz=0.115 0 0.007 rpy=-1.5708 0 0 -> xyz=0.115 0 0.007

Commit message: map update Nav2 error

File: ros_project_ws/src/qbot_description/urdf/qbot.urdf (robot description, URDF)
Before this commit: robot qbot, 10 links, 9 joints
Joints:
- joint base_joint: origin xyz=0 0 0.05 -> xyz=0 0 0.08
- joint wheel_left_joint: origin xyz=0 0.193 0.025 rpy=-1.5708 0 0 -> xyz=0 0.193 -0.03 rpy=-1.5708 0 0
- joint wheel_right_joint: origin xyz=0 -0.193 0.025 rpy=-1.5708 0 0 -> xyz=0 -0.193 -0.03 rpy=-1.5708 0 0

Commit message: SLAM mapping

File: ros_project_ws/src/qbot_description/urdf/qbot.urdf (robot description, URDF)
Before this commit: robot qbot, 10 links, 9 joints
Links:
- removed link lidar_link
- added link base_laser; visual cylinder length=0.05 radius=0.03

Commit message: URDF updated

File: ros_project_ws/src/qbot_description/urdf/qbot.urdf (robot description, URDF)
Before this commit: robot qbot, 10 links, 9 joints
Joints:
- joint lidar_joint: child lidar_link -> base_laser
